File: hardware/ArduinoMegaShield.sch (KiCad schematic (older format))
At the start: 34 parts, among them SW101 SW_Coded, SW102 SW_Coded, SW103 SW_Coded, U101 A4988, U102 A4988, U103 A4988

Commit message: changed dsub connectors to horizontal
Parts:
- SW101, SW102, SW103: MPN Copal S-1011A -> Copal S-1010A
Changed lines of the file:
@@
 F 3 "https://www.nidec-copal-electronics.com/e/catalog/switch/s-1000a&s-2000a.pdf" H 5055 2985 50  0001 C CNN
 F 4 "Value" H 5080 2960 60  0001 C CNN "Fieldname"
-F 5 "Copal S-1011A" H 5080 2960 60  0001 C CNN "MPN"
+F 5 "Copal S-1010A" H 5080 2960 60  0001 C CNN "MPN"
 	1    5080 2960
 	1    0    0    -1
@@
 F 3 "https://www.nidec-copal-electronics.com/e/catalog/switch/s-1000a&s-2000a.pdf" H 5120 5865 50  0001 C CNN
 F 4 "Value" H 5145 5840 60  0001 C CNN "Fieldname"
-F 5 "Copal S-1011A" H 5145 5840 60  0001 C CNN "MPN"
+F 5 "Copal S-1010A" H 5145 5840 60  0001 C CNN "MPN"
 	1    5145 5840
 	1    0    0    -1
@@
 F 3 "https://www.nidec-copal-electronics.com/e/catalog/switch/s-1000a&s-2000a.pdf" H 5105 4440 50  0001 C CNN
 F 4 "Value" H 5130 4415 60  0001 C CNN "Fieldname"
-F 5 "Copal S-1011A" H 5130 4415 60  0001 C CNN "MPN"
+F 5 "Copal S-1010A" H 5130 4415 60  0001 C CNN "MPN"
 	1    5130 4415
 	1    0    0    -1
